File: electronics/interior-lighting/interior-lighting.kicad_sch (KiCad schematic)
At the start: 48 parts, among them U1 APA102-2020, U10 APA102-2020, U11 APA102-2020, U12 APA102-2020, U13 APA102-2020, U14 APA102-2020, U15 APA102-2020, U16 APA102-2020, U17 APA102-2020, U18 APA102-2020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

Commit message: Internal lighting board finished
Parts:
- removed C1, C10, C16, C2, C22, C23, C24, C4: 100n_X7R_1005M, Applidyne_Capacitor:CAPC1005X60N, symbol appli_capacitor:100n_X7R_1005M
- added P1, P2, P3, P4, P5, P6: PAD_SOLDER_2mm, Applidyne_Connector:PAD_SOLDER_2mm_SQUARE, symbol appli_connector:PAD_SOLDER_2mm_SQUARE
- C11, C12, C13, C14, C15, C17, C18, C19, C20, C21, C3, C5, C6, C7, C8, C9: value 100n_X7R_1005M -> 100n_X7R_1608M; footprint Applidyne_Capacitor:CAPC1005X60N -> Applidyne_Capacitor:CAPC1608X90L; symbol appli_capacitor:100n_X7R_1005M -> appli_capacitor:100n_X7R_1608M; Supplier Part No 2210822 -> 2070398; Supplier Price 0.087 -> 0.011; Supplier Price Break 100 -> 1; Supplier URL http://au.element14.com/tdk/cga2b3x7r1h104k050bb/cap-mlcc-x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 -> http://au.element14.com/kemet/c0603c104k5racauto/cap-mlcc-x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; manf TDK -> KEMET; manf# CGA2B3X7R1H104K050BB -> C0603C104K5RACAUTO
Connections:
- net +3.3V: now also P4.1 (P1)
- net GND: now also P1.1 (P1)
- net at U24.1 (SDO): now also P5.1 (P1)
- net at U24.6 (CK0): now also P6.1 (P1)
- net at U1.2 (SDI): now also P3.1 (P1)
- net at U1.3 (CKI): now also P2.1 (P1)
Other:
- note added: "Just solder pads..."
- title: (none) -> SPE Tube Interior Lighting
- moved on the sheet: C11, C12, C13, C14, C15, C17, C18, C19, C20, C21, C5, C6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
