File: electronics/backplane/expansion.kicad_sch (KiCad schematic)
At the start: 17 parts, among them P1 JST_SH_4_RA, P10 CONN_01X03, P2 JST_SH_4_RA, P3 JST_SH_4_RA, P5 PAD_SOLDER_2mm, Q1 2N7002P

Commit message: Continue backplane design Cleanup schematic, most routing and placement done
Parts:
- removed SL2, SL3: SOLDER-LINK-2-TINY, Applidyne_Link:SJ1005-2N, symbol appli_link:SOLDER-LINK-2-TINY
- added D4, D5: BAV99, SOT23, symbol appli_device:BAV99
- added P5, P6, P7, P8 (x4): PAD_SOLDER_2mm, Applidyne_Connector:PAD_SOLDER_2mm, symbol appli_connector:PAD_SOLDER_2mm
- added R17, R18: 10R_1608M, Applidyne_Resistor:RESC1608X50N, symbol appli_resistor:10R_1608M
Connections:
- net +3.3V: now also D4.2 (C2), D5.2 (C2), P8.1 (P1)
- net +POWER: now also P8.1 (P1)
- net CIPO: now also P6.1 (P1)
- net CLK: now also P5.1 (P1)
- net COPI: now also P7.1 (P1)
- net GND: now also D4.1 (A1), D5.1 (A1), P8.1 (P1)
- net ~{CS}: now also P8.1 (P1)
- new net ANALOG_IN: D5.3, R18.1
- new net DIGITAL_OUT: D4.3, R17.1
Other:
- note added: "CHECK PROCESSOR SUPPORT IF UNSUPPORTED, CONSIDER MERGE BRIDGES"
- note added: "Most MicroMod Processors don't connect SPI1. These pads allow for expansion/bodge wires."
- note added: "SPARE IO"
- note added: "SPI1 BREAKOUT"
- note removed: "Allows other I2C connectors to be used when the processor board only implements one I2C channel."
- note removed: "CHECK PROCESSOR SUPPORT"
- note removed: "GPIO"
- note removed: "I2C BUS MERGE"
- note removed: "SPI Header?"
- note removed: "TODO: Consider installing RA"
- note removed: "TX2 seems to be rarely available with current MicroMod processor implementations"
- moved on the sheet: D1, F2, P10, Q1, R13, R8, R9

Commit message: Continued routing Labels, most traces, most pours
Parts:
- removed D4, D5: BAV99, SOT23, symbol appli_device:BAV99
- removed R17, R18: 10R_1608M, Applidyne_Resistor:RESC1608X50N, symbol appli_resistor:10R_1608M

Commit message: Backplane routing complete General schematic cleanup, board cosmetics etc
Parts:
- added P8 (x2): PAD_SOLDER_2mm, Applidyne_Connector:PAD_SOLDER_2mm, symbol appli_connector:PAD_SOLDER_2mm
Connections:
- net ANALOG_IN: now also P8.1 (P1)
- net DIGITAL_OUT: now also P8.1 (P1)
Other:
- company: (none) -> Check processor support before use!
- title: (none) -> Expansion IO
- moved on the sheet: D1, F2, P10, P5, P6, P7, P8, Q1, R13, R8, R9

Commit message: Fixed backplane i2c connector 3D model/footprint linkage Also minor schematic cleanup
Changed lines of the file:
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@@
-    )
-  )
-  (symbol (lib_id "appli_power:+3.3V") (at 106.68 62.23 0) (unit 1)
-    (in_bom yes) (on_board yes) (dnp no) (fields_autoplaced)
-    (property "Reference" "#PWR026" (at 106.68 66.04 0)
-      (effects (font (size 1.27 1.27)) hide)
-    )
-    (property "Value" "+3.3V" (at 106.68 57.15 0)
-      (effects (font (size 1.27 1.27)))
-    )
-    (property "Footprint" "" (at 106.68 62.23 0)
-      (effects (font (size 1.27 1.27)) hide)
-    )
-    (property "Datasheet" "" (at 106.68 62.23 0)
-      (effects (font (size 1.27 1.27)) hide)
-    )
-    (pin "1")
-    (instances
-      (project "backplane"
-        (path "/0bfdf1e4-b99d-46d4-adfc-42d352d37946/86d6522f-71ec-4ba6-99bb-080f48f086cd"
-          (reference "#PWR026") (unit 1)
-        )
-      )
     )
   )
